File: RoRoR/02_Assemble/RoRoR.kicad_pcb (KiCad board)
At the start: 2 copper layers, 304.4 x 98.8 mm, 135 parts, among them J1 Conn_01x02, SW1 SW_PUSH, SW10 SW_PUSH, SW11 SW_PUSH, SW12 SW_PUSH, SW13 SW_PUSH, SW14 SW_PUSH, SW15 SW_PUSH, SW16 SW_PUSH, SW17 SW_PUSH, SW18 SW_PUSH, SW19 SW_PUSH, SW2 SW_PUSH, SW20 SW_PUSH, SW21 SW_PUSH, SW22 SW_PUSH, SW23 SW_PUSH, SW24 SW_PUSH, SW25 SW_PUSH, SW26 SW_PUSH, SW27 RotaryEncoder_Switch, SW28 SW_PUSH, SW29 SW_PUSH, SW3 SW_PUSH, SW30 SW_PUSH, SW31 SW_PUSH, SW32 SW_PUSH, SW33 SW_PUSH, SW34 SW_PUSH, SW35 SW_PUSH, SW36 SW_PUSH, SW37 SW_PUSH, SW38 SW_PUSH, SW39 SW_PUSH, SW4 SW_PUSH, SW40 SW_PUSH, SW41 SW_PUSH, SW42 SW_PUSH, SW43 SW_PUSH, SW44 SW_PUSH, SW45 SW_PUSH, SW46 SW_PUSH, SW47 SW_PUSH, SW48 SW_PUSH, SW49 SW_PUSH, SW5 SW_PUSH, SW50 SW_PUSH, SW51 SW_PUSH, SW52 SW_PUSH, SW53 SW_PUSH, SW54 RotaryEncoder_Switch, SW55 SW_PUSH, SW6 SW_PUSH, SW7 SW_PUSH, SW8 SW_PUSH, SW9 SW_PUSH, U1 BLEMicroPro

Commit message: update
Routing:
- net GND: track 594.2 -> 557.2 mm
- net VCC: track 454.6 -> 441.1 mm
- net Col2: track 393.5 -> 385.6 mm
- net Col0: track 425.9 -> 418.1 mm
- net Col3: track 388.2 -> 381.1 mm
- net Net-(D32-Pad1): track 21.3 -> 16.9 mm
- net Row3: track 392.1 -> 389.0 mm
- net Net-(D22-Pad2): track 16.6 -> 14.1 mm
- net Col1: track 404.3 -> 401.9 mm
- net Net-(D53-Pad1): track 35.1 -> 32.8 mm
- net Net-(L21-Pad1): track 40.0 -> 38.0 mm, vias 3 -> 2
- net Net-(L22-Pad1): track 21.1 -> 19.4 mm
- net Net-(D48-Pad1): track 18.1 -> 16.9 mm
- net Net-(D44-Pad1): track 18.1 -> 16.9 mm
- net Net-(D40-Pad1): track 18.1 -> 16.9 mm
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