File: RoSoR/01_Top_TH_hole/RoSoR.kicad_pcb (KiCad board)
At the start: 2 copper layers, 314.4 x 98.8 mm, 70 parts, among them J10 Conn_01x01, J11 Conn_01x01, J12 Conn_01x01, J13 Conn_01x01, J14 Conn_01x01, J15 Conn_01x01, J16 Conn_01x01, J17 Conn_01x01, J2 Conn_01x01, J3 Conn_01x01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

Commit message: update
Routing:
- added copper zone on F.Cu, net (none)
Other:
- outline, holes or cut-outs redrawn
