File: RoSoR/02_Assemble/RoSoR.kicad_pcb (KiCad board)
At the start: 2 copper layers, 304.4 x 98.8 mm, 135 parts, among them J1 Conn_01x02, SW1 SW_PUSH, SW10 SW_PUSH, SW11 SW_PUSH, SW12 SW_PUSH, SW13 SW_PUSH, SW14 SW_PUSH, SW15 SW_PUSH, SW16 SW_PUSH, SW17 SW_PUSH, SW18 SW_PUSH, SW19 SW_PUSH, SW2 SW_PUSH, SW20 SW_PUSH, SW21 SW_PUSH, SW22 SW_PUSH, SW23 SW_PUSH, SW24 SW_PUSH, SW25 SW_PUSH, SW26 SW_PUSH, SW27 RotaryEncoder_Switch, SW28 SW_PUSH, SW29 SW_PUSH, SW3 SW_PUSH, SW30 SW_PUSH, SW31 SW_PUSH, SW32 SW_PUSH, SW33 SW_PUSH, SW34 SW_PUSH, SW35 SW_PUSH, SW36 SW_PUSH, SW37 SW_PUSH, SW38 SW_PUSH, SW39 SW_PUSH, SW4 SW_PUSH, SW40 SW_PUSH, SW41 SW_PUSH, SW42 SW_PUSH, SW43 SW_PUSH, SW44 SW_PUSH, SW45 SW_PUSH, SW46 SW_PUSH, SW47 SW_PUSH, SW48 SW_PUSH, SW49 SW_PUSH, SW5 SW_PUSH, SW50 SW_PUSH, SW51 SW_PUSH, SW52 SW_PUSH, SW53 SW_PUSH, SW54 RotaryEncoder_Switch, SW55 SW_PUSH, SW6 SW_PUSH, SW7 SW_PUSH, SW8 SW_PUSH, SW9 SW_PUSH, U1 BLEMicroPro

Commit message: fix
Parts:
- added G***: LOGO, LOGO, F.Cu at (38.1, 28.6)
Other:
- board text added: "RoSoR Rev1.0 2022/2/22 52Keys+2Rotary encoders Ortholinear Keyboard"
- board text removed: "RoRoR Rev1.0 2022/2/18 52Keys+2Rotary encoders Ortholinear Keyboard"

Commit message: update
Other:
- board text added: "RoSoR Rev1.0 For GL516 Designed by Takamegane Date:2022/2/22 52Keys+2Rotary encoders Ortholinear Keyboard"
- board text removed: "RoSoR Rev1.0 2022/2/22 52Keys+2Rotary encoders Ortholinear Keyboard"

Commit message: update
Parts:
- added G***: LOGO, LOGO, B.Cu at (31.4, 33.3)
Changed lines of the file:
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@@
     )
+  )
+  (footprint "LOGO" (layer "B.Cu")
+    (at 31.402708 33.337472 -150)
+    (attr board_only exclude_from_pos_files exclude_from_bom)
+    (fp_text reference "G***" (at 0 0 30) (layer "F.Fab")
+      (effects (font (size 1.524 1.524) (thickness 0.3)))
+    )
+    (fp_text value "LOGO" (at 0.75 0 30) (layer "F.Fab") hide
+      (effects (font (size 1.524 1.524) (thickness 0.3)))
+    )
+    (fp_poly (pts
+        (xy -2.305506 1.888189)
+        (xy -1.632727 1.805339)
+        (xy -0.857193 1.672312)
+        (xy -0.729074 1.648003)
+        (xy -0.31636 1.578072)
+        (xy 0.006223 1.555398)
+        (xy 0.330664 1.579981)
+        (xy 0.729074 1.648003)
+        (xy 1.525611 1.788848)
+        (xy 2.209409 1.878887)
+        (xy 2.84765 1.922351)
+        (xy 3.507513 1.923474)
+        (xy 4.256179 1.88649)
+        (xy 4.379115 1.878001)
+        (xy 4.879694 1.836474)
+        (xy 5.317924 1.788907)
+        (xy 5.657302 1.740117)
+        (xy 5.861325 1.694921)
+        (xy 5.89873 1.677481)
+        (xy 5.996776 1.49091)
+        (xy 6.016142 1.213935)
+        (xy 5.961199 0.924982)
+        (xy 5.844892 0.711619)
+        (xy 5.721117 0.515774)
+        (xy 5.586202 0.214181)
+        (xy 5.501298 -0.02815)
+        (xy 5.348801 -0.437832)
+        (xy 5.14876 -0.868844)
+        (xy 5.042147 -1.062965)
+        (xy 4.849563 -1.355469)
+        (xy 4.66262 -1.535444)
+        (xy 4.409296 -1.66173)
+        (xy 4.233334 -1.723758)
+        (xy 3.811207 -1.82338)
+        (xy 3.297809 -1.885434)
+        (xy 2.757255 -1.907899)
+        (xy 2.253659 -1.888754)
+        (xy 1.851137 -1.825977)
+        (xy 1.768591 -1.801453)
+        (xy 1.373367 -1.579494)
+        (xy 1.025453 -1.196361)
+        (xy 0.715922 -0.641293)
+        (xy 0.619987 -0.416837)
+        (xy 0.452089 -0.003998)
+        (xy 0.333134 0.264839)
+        (xy 0.242639 0.420541)
+        (xy 0.160119 0.493977)
+        (xy 0.065089 0.516013)
+        (xy 0 0.517407)
+        (xy -0.111037 0.510373)
+        (xy -0.198165 0.468619)
+        (xy -0.281991 0.361167)
+        (xy -0.383121 0.157042)
+        (xy -0.522163 -0.174735)
+        (xy -0.617357 -0.410649)
+        (xy -0.901338 -1.008027)
+        (xy -1.20687 -1.432291)
+        (xy -1.54529 -1.6982)
+        (xy -1.641904 -1.743985)
+        (xy -2.058209 -1.857763)
+        (xy -2.590513 -1.916221)
+        (xy -3.173634 -1.91478)
+        (xy -3.556853 -1.878496)
+        (xy -4.11201 -1.765196)
+        (xy -4.547775 -1.578236)
+        (xy -4.890853 -1.291949)
+        (xy -5.167951 -0.880672)
+        (xy -5.405776 -0.318739)
+        (xy -5.509532 -0.00197)
+        (xy -5.62928 0.322551)
+        (xy -5.765176 0.597182)
+        (xy -5.844891 0.711619)
+        (xy -5.966055 0.939794)
+        (xy -6.017043 1.230121)
+        (xy -5.993484 1.504175)
+        (xy -5.89873 1.677481)
+        (xy -5.765527 1.719585)
+        (xy -5.480972 1.767392)
+        (xy -5.081569 1.816088)
+        (xy -4.60382 1.860855)
+        (xy -4.379114 1.878001)
+        (xy -3.61152 1.920287)
+        (xy -2.94271 1.925094)
+      ) (layer "B.SilkS") (width 0) (fill solid))
   )
   (gr_poly
@@
       (xy 171.45 79.208605)
     ) (layer "F.SilkS") (width 0.45) (fill none))
-  (gr_circle (center 154.78125 95.25) (end 167.878125 95.25) (layer "F.SilkS") (width 0.15) (fill none))
+  (gr_circle (center 154.78125 95.25) (end 167.878125 95.25) (layer "F.SilkS") (width 0.25) (fill none))
   (gr_circle (center 188.11875 95.25) (end 198.834375 95.25) (layer "F.SilkS") (width 0.45) (fill none))
-  (gr_circle (center 188.11875 95.25) (end 197.64375 95.25) (layer "F.SilkS") (width 0.45) (fill none))
-  (gr_circle (center 154.78125 95.25) (end 164.380376 95.25) (layer "F.SilkS") (width 0.45) (fill none))
-  (gr_circle (center 154.78125 95.25) (end 165.496875 95.25) (layer "F.SilkS") (width 0.35) (fill none))
+  (gr_circle (center 188.11875 95.25) (end 197.64375 95.25) (layer "F.SilkS") (width 0.5) (fill none))
+  (gr_circle (center 154.78125 95.25) (end 164.380376 95.25) (layer "F.SilkS") (width 0.5) (fill none))
+  (gr_circle (center 154.78125 95.25) (end 165.496875 95.25) (layer "F.SilkS") (width 0.45) (fill none))
   (gr_circle (center 188.11875 95.25) (end 201.215625 95.25) (layer "F.SilkS") (width 0.25) (fill none))
   (gr_poly
@@
     ) (layer "F.SilkS") (width 0.35) (fill none))
   (gr_circle (center 188.11875 95.25) (end 200.084383 95.25) (layer "F.SilkS") (width 0.35) (fill none))
-  (gr_circle (center 154.78125 95.25) (end 166.6875 95.25) (layer "F.SilkS") (width 0.25) (fill none))
+  (gr_circle (center 154.78125 95.25) (end 166.6875 95.25) (layer "F.SilkS") (width 0.35) (fill none))
   (gr_poly
     (pts

Commit message: update
Other:
- board text added: "RoSoR for GL516 Rev1.0 52Keys+2Rotary encoders Ortholinear Keyboard Designed by Takamegane Date:2022/2/22"
- board text removed: "RoSoR Rev1.0 For GL516 Designed by Takamegane Date:2022/2/22 52Keys+2Rotary encoders Ortholinear Keyboard"
